File: Hardware/Eagle_Version/MAKKI_ISMAIL_ESPS3_CAM/MAKKI_ISMAIL_ESPS3_CAM/MAKKI_ISMAIL_ESPS3_CAM.sch (EAGLE design)
At the start: 76 parts, among them IC1 LC709203F/MH, IC2 ESP32-S3-WROOM-1-N16R8, IC3 XC6206P282MR-G, IC4 ICS-43434, J1 2-2328702-4, J2 B2B-XH-A, Q1 DMG3415U, Q2 2N7002, Q3 DMG3415U, SW1 KMR2, SW2 KMR2, U1 MAX98357A, U2 AP2112/RT9080-3.3, U3 MCP73831T-2ACI/OT, X1 JSTPH, X3 USB C

Commit message: Version Corrige
Parts:
- removed D3: RED, microbuilder:LED0603_NOOUTLINE
- removed JP1: (no value), microbuilder:HEADER-1X7THICKER
- removed R10: 5.1K, microbuilder:RESISTOR_0603_NOOUT
Connections:
- removed net 1.8V: IC2.IO48
- removed net D13: R10.1
- removed net D8: IC2.IO10, J1.14
- removed net D9: IC2.IO12, J1.12
- removed net N$5: D3.A, R10.2
- removed net RX: IC2.IO38, JP1.4
- removed net TX: IC2.IO39, JP1.5
- net D7: now also IC2.IO38; no longer IC2.IO9
- net GND: no longer D3.C
- net RESET: no longer J1.6
- net RXD0: no longer JP1.6
- net TXD0: no longer JP1.7
- net XVCLK: now also IC2.IO39; no longer IC2.IO11
Changed lines of the file:
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@@
 <part name="SW2" library="microbuilder" deviceset="SWITCH_TACT_SMT" device="4.6X2.8" override_package3d_urn="urn:adsk.eagle:package:51317600/2" override_package_urn="urn:adsk.eagle:footprint:51317601/1" value="KMR2"/>
 <part name="GND6" library="supply1" library_urn="urn:adsk.eagle:library:371" deviceset="GND" device=""/>
-<part name="D3" library="microbuilder" deviceset="LED" device="0603_NOOUTLINE" override_package3d_urn="urn:adsk.eagle:package:51321308/2" override_package_urn="urn:adsk.eagle:footprint:51321309/1" value="RED"/>
-<part name="R10" library="microbuilder" deviceset="RESISTOR" device="_0603_NOOUT" override_package3d_urn="urn:adsk.eagle:package:51321310/2" override_package_urn="urn:adsk.eagle:footprint:51321311/1" value="5.1K"/>
 <part name="U$10" library="microbuilder" deviceset="3.3V" device=""/>
 <part name="C2" library="microbuilder" deviceset="CAP_CERAMIC" device="0805-NOOUTLINE" override_package3d_urn="urn:adsk.eagle:package:51317638/2" override_package_urn="urn:adsk.eagle:footprint:51317639/1" value="10uF"/>
@@
 <part name="U$2" library="microbuilder" deviceset="3.3V" device=""/>
 <part name="U$4" library="microbuilder" deviceset="GND" device=""/>
-<part name="U$8" library="microbuilder" deviceset="GND" device=""/>
 <part name="Q3" library="microbuilder" deviceset="MOSFET-P" device="" override_package3d_urn="urn:adsk.eagle:package:51317626/2" override_package_urn="urn:adsk.eagle:footprint:51317627/1" value="DMG3415U"/>
 <part name="R12" library="microbuilder" deviceset="RESISTOR" device="_0603_NOOUT" override_package3d_urn="urn:adsk.eagle:package:51317881/2" override_package_urn="urn:adsk.eagle:footprint:51317882/1" value="100K"/>
@@
 <part name="U$63" library="microbuilder" deviceset="3.3V" device=""/>
 <part name="J2" library="Connector" library_urn="urn:adsk.eagle:library:16378166" deviceset="B2B-XH-A" device="" package3d_urn="urn:adsk.eagle:package:24957641/7"/>
-<part name="JP1" library="microbuilder" deviceset="HEADER-1X7" device="THICKER"/>
 <part name="TP2" library="microbuilder" deviceset="TESTPOINT" device="ROUND1.5MMNO"/>
 <part name="TP3" library="microbuilder" deviceset="TESTPOINT" device="ROUND1.5MMNO"/>
@@
 <attribute name="VALUE" x="121.92" y="134.62" size="1.778" layer="96"/>
 </instance>
-<instance part="D3" gate="G$1" x="111.76" y="33.02" smashed="yes" rot="R90">
-<attribute name="NAME" x="107.315" y="31.75" size="1.27" layer="95" rot="R90" align="center"/>
-<attribute name="VALUE" x="114.554" y="31.75" size="1.27" layer="96" rot="R90" align="center"/>
-</instance>
-<instance part="R10" gate="G$1" x="111.76" y="22.86" smashed="yes" rot="R90">
-<attribute name="NAME" x="109.22" y="22.86" size="1.27" layer="95" font="vector" rot="R90" align="center"/>
-<attribute name="VALUE" x="111.76" y="22.86" size="1.016" layer="96" font="vector" ratio="15" rot="R90" align="center"/>
-</instance>
 <instance part="U$10" gate="G$1" x="63.5" y="162.56" smashed="yes">
 <attribute name="VALUE" x="61.976" y="163.576" size="1.27" layer="96"/>
@@
 <instance part="U$4" gate="G$1" x="101.6" y="139.7" smashed="yes">
 <attribute name="VALUE" x="100.076" y="137.16" size="1.27" layer="96"/>
-</instance>
-<instance part="U$8" gate="G$1" x="114.3" y="40.64" smashed="yes" rot="R90">
-<attribute name="VALUE" x="116.84" y="39.116" size="1.27" layer="96" rot="R90"/>
 </instance>
 <instance part="Q3" gate="G$1" x="25.4" y="162.56" smashed="yes" rot="MR180">
@@
 <pinref part="C1" gate="G$1" pin="2"/>
 <pinref part="U$4" gate="G$1" pin="GND"/>
-</segment>
-<segment>
-<pinref part="U$8" gate="G$1" pin="GND"/>
-<pinref part="D3" gate="G$1" pin="C"/>
-<wire x1="111.76" y1="35.56" x2="111.76" y2="40.64" width="0.1524" layer="91"/>
 </segment>
 <segment>
@@
 <pinref part="TP3" gate="G$1" pin="P$1"/>
 </segment>
-<segment>
-<pinref part="J1" gate="G$1" pin="6"/>
-<wire x1="99.314" y1="76.2" x2="109.474" y2="76.2" width="0.1524" layer="91"/>
-<label x="101.854" y="76.2" size="1.778" layer="95"/>
-</segment>
 </net>
 <net name="EN" class="0">
@@
 </segment>
 </net>
-<net name="N$5" class="0">
-<segment>
-<pinref part="R10" gate="G$1" pin="2"/>
-<pinref part="D3" gate="G$1" pin="A"/>
-</segment>
-</net>
 <net name="D+" class="0">
 <segment>
@@
 </segment>
 </net>
-<net name="D9" class="0">
-<segment>
-<pinref part="J1" gate="G$1" pin="12"/>
-<wire x1="99.314" y1="91.44" x2="109.474" y2="91.44" width="0.1524" layer="91"/>
-<label x="101.854" y="91.44" size="1.778" layer="95"/>
-</segment>
-<segment>
-<pinref part="IC2" gate="G$1" pin="IO12"/>
-<wire x1="20.32" y1="68.58" x2="7.62" y2="68.58" width="0.1524" layer="91"/>
-<label x="12.7" y="68.58" size="1.778" layer="95"/>
-</segment>
-</net>
-<net name="D13" class="0">
-<segment>
-<pinref part="R10" gate="G$1" pin="1"/>
-<wire x1="111.76" y1="17.78" x2="111.76" y2="7.62" width="0.1524" layer="91"/>
-<label x="111.76" y="10.16" size="1.778" layer="95" rot="R90"/>
-</segment>
-</net>
 <net name="D5" class="0">
 <segment>
@@
 <wire x1="20.32" y1="96.52" x2="7.62" y2="96.52" width="0.1524" layer="91"/>
 <label x="12.7" y="96.52" size="1.778" layer="95"/>
-</segment>
-</net>
-<net name="RX" class="0">
-<segment>
-<pinref part="IC2" gate="G$1" pin="IO38"/>
-<wire x1="53.34" y1="104.14" x2="66.04" y2="104.14" width="0.1524" layer="91"/>
-<label x="55.88" y="104.14" size="1.778" layer="95"/>
-</segment>
-</net>
-<net name="TX" class="0">
-<segment>
-<pinref part="IC2" gate="G$1" pin="IO39"/>
-<wire x1="53.34" y1="101.6" x2="66.04" y2="101.6" width="0.1524" layer="91"/>
-<label x="55.88" y="101.6" size="1.778" layer="95"/>
 </segment>
 </net>
@@
 </segment>
 <segment>
-<pinref part="IC2" gate="G$1" pin="IO11"/>
-<wire x1="20.32" y1="71.12" x2="7.62" y2="71.12" width="0.1524" layer="91"/>
-<label x="10.16" y="71.12" size="1.778" layer="95"/>
-</segment>
-</net>
-<net name="D8" class="0">
-<segment>
-<pinref part="J1" gate="G$1" pin="14"/>
-<wire x1="99.314" y1="96.52" x2="109.474" y2="96.52" width="0.1524" layer="91"/>
-<label x="101.854" y="96.52" size="1.778" layer="95"/>
-</segment>
-<segment>
-<pinref part="IC2" gate="G$1" pin="IO10"/>
-<wire x1="20.32" y1="73.66" x2="7.62" y2="73.66" width="0.1524" layer="91"/>
-<label x="12.7" y="73.66" size="1.778" layer="95"/>
+<pinref part="IC2" gate="G$1" pin="IO39"/>
+<wire x1="53.34" y1="101.6" x2="66.04" y2="101.6" width="0.1524" layer="91"/>
+<label x="55.88" y="101.6" size="1.778" layer="95"/>
 </segment>
 </net>
@@
 </segment>
 <segment>
-<pinref part="IC2" gate="G$1" pin="IO9"/>
-<wire x1="20.32" y1="76.2" x2="7.62" y2="76.2" width="0.1524" layer="91"/>
-<label x="12.7" y="76.2" size="1.778" layer="95"/>
+<pinref part="IC2" gate="G$1" pin="IO38"/>
+<wire x1="53.34" y1="104.14" x2="66.04" y2="104.14" width="0.1524" layer="91"/>
+<label x="55.88" y="104.14" size="1.778" layer="95"/>
 </segment>
 </net>
@@
 <wire x1="20.32" y1="63.5" x2="7.62" y2="63.5" width="0.1524" layer="91"/>
 <label x="12.7" y="63.5" size="1.778" layer="95"/>
-</segment>
-</net>
-<net name="1.8V" class="0">
-<segment>
-<pinref part="IC2" gate="G$1" pin="IO48"/>
-<wire x1="20.32" y1="55.88" x2="7.62" y2="55.88" width="0.1524" layer="91"/>
-<label x="12.7" y="55.88" size="1.778" layer="95"/>
-</segment>
-</net>
-<net name="N$16" class="0">
-<segment>
-<wire x1="137.16" y1="58.42" x2="132.08" y2="58.42" width="0.1524" layer="91"/>
 </segment>
 </net>
@@
 <attribute name="VALUE" x="66.04" y="48.26" size="1.778" layer="96" rot="R180" align="bottom-center"/>
 </instance>
-<instance part="JP1" gate="A" x="160.02" y="50.8" smashed="yes">
-<attribute name="NAME" x="153.67" y="61.595" size="1.778" layer="95"/>
-<attribute name="VALUE" x="153.67" y="38.1" size="1.778" layer="96"/>
-</instance>
 <instance part="TP4" gate="G$1" x="58.42" y="132.08" smashed="yes" rot="R270">
 <attribute name="NAME" x="64.008" y="132.08" size="1.27" layer="95" align="center-left"/>
@@
 </segment>
 </net>
-<net name="TXD0" class="0">
-<segment>
-<pinref part="JP1" gate="A" pin="7"/>
-<wire x1="157.48" y1="43.18" x2="147.32" y2="43.18" width="0.1524" layer="91"/>
-<label x="149.86" y="43.18" size="1.778" layer="95"/>
-</segment>
-</net>
-<net name="RXD0" class="0">
-<segment>
-<pinref part="JP1" gate="A" pin="6"/>
-<wire x1="157.48" y1="45.72" x2="147.32" y2="45.72" width="0.1524" layer="91"/>
-<label x="149.86" y="45.72" size="1.778" layer="95"/>
-</segment>
-</net>
-<net name="TX" class="0">
-<segment>
-<pinref part="JP1" gate="A" pin="5"/>
-<wire x1="157.48" y1="48.26" x2="147.32" y2="48.26" width="0.1524" layer="91"/>
-<label x="149.86" y="48.26" size="1.778" layer="95"/>
-</segment>
-</net>
-<net name="RX" class="0">
-<segment>
-<pinref part="JP1" gate="A" pin="4"/>
-<wire x1="157.48" y1="50.8" x2="147.32" y2="50.8" width="0.1524" layer="91"/>
-<label x="149.86" y="50.8" size="1.778" layer="95"/>
-</segment>
-</net>
